File: hardware/led-driver/led-driver.kicad_pcb (KiCad board)
At the start: 2 copper layers, 291.5 x 19.7 mm, 63 parts, among them J1 Conn_01x04_Male, J2 Conn_01x04_Male, U1 PCA9634, U2 PCA9634, U3 PCA9634

Commit message: Narrower board: remove explicit ground trace, use fill.
Routing:
- net GND: track 378.4 -> 51.4 mm, vias 32 -> 149
Other:
- board size 291.5 x 19.7 mm -> 291.6 x 18.3 mm

Commit message: Improve board, move to KiCad 6.
Parts:
- C1, C2, C3, C4: footprint Capacitors_SMD:C_0805_HandSoldering -> Capacitor_SMD:C_0805_2012Metric_Pad1.18x1.45mm_HandSolder
- DA-0, DA-1, DA-2, DA-3, DA-4, DA-5, DA-6, DA-7, DA-P1, DB-0, DB-1, DB-2, DB-3, DB-4, DB-5, DB-6, DB-7, DB-P1, DX-0, DX-1, DX-2, DX-3, DX-4, DX-5: footprint LEDs:LED_D3.0mm -> Library:LED_D3.0mm-nosilk
- J1, J2: footprint Socket_Strips:Socket_Strip_Straight_1x04_Pitch2.54mm -> Library:PinHeader_1x04_P2.54mm_Vertical_mirrored
- JP1, JP3: footprint SparkFun:SMT-JUMPER_3_NO_SILK -> Jumper:SolderJumper-3_P1.3mm_Open_RoundedPad1.0x1.5mm_NumberLabels
- JP2: value A2 -> A5; footprint SparkFun:SMT-JUMPER_3_NO_SILK -> Jumper:SolderJumper-3_P1.3mm_Open_RoundedPad1.0x1.5mm_NumberLabels
- JP4: value A1 -> A6; footprint SparkFun:SMT-JUMPER_3_NO_SILK -> Jumper:SolderJumper-3_P1.3mm_Open_RoundedPad1.0x1.5mm_NumberLabels
- R1, R10, R11, R12, R13, R14, R15, R16, R17, R18, R19, R2, R20, R21, R22, R23, R24, R3, R4, R5, R6, R7, R8, R9: footprint Resistors_SMD:R_0805_HandSoldering -> Resistor_SMD:R_0805_2012Metric_Pad1.20x1.40mm_HandSolder
- U1, U2, U3: footprint Housings_SOIC:SOIC-20W_7.5x12.8mm_Pitch1.27mm -> Package_SO:SOIC-20W_7.5x12.8mm_P1.27mm
- moved JP4 125.5 mm to (98.6, 23.4)
- moved JP2 121.9 mm to (101.9, 23.4)
- moved JP3 114.6 mm to (105.3, 23.4)
- moved JP1 111.6 mm to (108.7, 23.4)
- moved U2 97.5 mm to (140.3, 23.2)
- moved C2 96.9 mm to (148.6, 23.5)
- moved U3 74.7 mm to (178.4, 23.2)
- moved C3 74.1 mm to (186.7, 23.5)
- moved J1 58.6 mm to (206.5, 27.4), turned to 90 degrees
- moved C1 55.6 mm to (64.8, 21.3)
- moved U1 54.8 mm to (56.4, 21.1)
- moved H1 45.0 mm to (225.6, 24.9)
- moved J2 31.6 mm to (20.3, 27.4), turned to 90 degrees
- moved H2 28.7 mm to (13.2, 24.9)
- moved R8 5.27 mm to (105.2, 12.7), turned to 0 degrees
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Routing:
- net /A6: track 269.3 -> 131.4 mm
- net /A3: track 264.5 -> 131.0 mm
- net /A5: track 263.9 -> 131.5 mm
- net /A4: track 261.1 -> 130.2 mm
- net Net-(R9-Pad2): track 115.8 -> 23.6 mm
- net /SDA: track 296.6 -> 205.6 mm
- net Net-(R10-Pad2): track 107.2 -> 20.5 mm
- net Net-(R22-Pad2): track 88.3 -> 3.06 mm, vias 2 -> 0
- net +5V: track 339.6 -> 419.8 mm, vias 7 -> 20
- net Net-(R21-Pad2): track 103.2 -> 24.1 mm
- net /SCL: track 287.4 -> 208.4 mm
- net Net-(R11-Pad2): track 90.0 -> 17.9 mm
- net Net-(R17-Pad2): track 142.8 -> 75.1 mm
- net Net-(R20-Pad2): track 104.7 -> 38.4 mm
- net Net-(R19-Pad2): track 115.0 -> 51.4 mm
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Other:
- board size 291.6 x 18.3 mm -> 221.5 x 18.3 mm
- net class Default removed
- board text added: "System/360 Model 50 console LED driver Ken Shirriff righto.com/s360 v1.0"
- board text removed: "System/360 Model 50 console driver Ken Shirriff righto.com/s360"
- board text removed: "v1.0"

Commit message: Submitted version of board, 1.2.1
Parts:
- removed DA-P1, DB-7, DB-P1, DX-0, DX-1, DX-2, DX-3, DX-4, DX-5: LED, Library:LED_D3.0mm-nosilk
- added C1: .33uF, Capacitor_SMD:C_0805_2012Metric_Pad1.18x1.45mm_HandSolder, F.Cu at (67.8, 60.3)
- added C11: .33uF, Capacitor_SMD:C_0805_2012Metric_Pad1.18x1.45mm_HandSolder, F.Cu at (91.8, 60.4)
- added C12: 100uF, Capacitor_Tantalum_SMD:CP_EIA-7343-40_Kemet-Y_Pad2.25x2.55mm_HandSolder, F.Cu at (42.2, 48.9)
- added C5: .33uF, Capacitor_SMD:C_0805_2012Metric_Pad1.18x1.45mm_HandSolder, F.Cu at (227.2, 39.2)
- added C6: .33uF, Capacitor_SMD:C_0805_2012Metric_Pad1.18x1.45mm_HandSolder, F.Cu at (228.3, 58.0)
- added C8: .33uF, Capacitor_SMD:C_0805_2012Metric_Pad1.18x1.45mm_HandSolder, F.Cu at (228.3, 49.9)
- added C9: .33uF, Capacitor_SMD:C_0805_2012Metric_Pad1.18x1.45mm_HandSolder, F.Cu at (229.1, 69.8)
- added D0: LED, Library:LED_D3.0mm-nosilk, F.Cu at (29.5, 26.9)
- added DP0: LED, Library:LED_D3.0mm-nosilk, F.Cu at (131.1, 26.9)
- added DP1: LED, Library:LED_D3.0mm-nosilk, F.Cu at (245.4, 26.9)
- added J3: Conn_02x20_Odd_Even, Samtec:SAMTEC_TSS-120-04-F-D-RA-mirror, F.Cu at (110.0, 69.9)
- added J4: Conn_02x25_Odd_Even, Samtec:SAMTEC_TSS-125-04-F-D-RA-mirror, F.Cu at (198.7, 69.8)
- added J5: Conn_01x02, Samtec:SAMTEC_TSS-102-04-F-S-RA, F.Cu at (236.2, 72.4)
- added J6: Conn_01x05, Samtec:SAMTEC_TSS-105-04-F-S-RA, F.Cu at (130.4, 72.4)
- added J7: Conn_02x10_Odd_Even, Samtec:SAMTEC_TSS-110-04-F-D-RA-mirror, F.Cu at (234.8, 35.5)
- added J8: Conn_01x02_Male, Samtec:SAMTEC_TSS-102-04-F-S-RA, F.Cu at (226.3, 72.4)
- added J9: Conn_01x02_Male, Samtec:SAMTEC_TSS-102-04-F-S-RA, F.Cu at (57.1, 72.4)
- added L1: 330 µH, Library:L_Bourns_SDR1307, F.Cu at (33.2, 60.6)
- added L2: 330 µH, Library:L_Bourns_SDR1307, F.Cu at (54.0, 60.7)
- added R25: 4.7K, Resistor_SMD:R_0805_2012Metric_Pad1.20x1.40mm_HandSolder, F.Cu at (233.7, 67.0)
- added U4: PCA9555D, Package_SO:SOIC-24W_7.5x15.4mm_P1.27mm, F.Cu at (77.1, 60.1)
- added U5: ADS7828, Package_SO:TSSOP-16_4.4x5mm_P0.65mm, F.Cu at (229.1, 43.2)
- added U6: ADS7828, Package_SO:TSSOP-16_4.4x5mm_P0.65mm, F.Cu at (228.5, 53.9)
- added U7: MCP47CVB01, Package_SO:MSOP-10_3x3mm_P0.5mm, F.Cu at (227.8, 66.8)
- added U8: PCA9555D, Package_SO:SOIC-24W_7.5x15.4mm_P1.27mm, F.Cu at (100.8, 60.1)
- C10: renamed from C3; value .1uF -> .33uF
- C3: renamed from C1; value .1uF -> .33uF
- C4: value 10uF -> .33uF
- C7: renamed from C2; value .1uF -> .33uF
- H1, H2: footprint Mounting_Holes:MountingHole_4.3mm_M4 -> MountingHole:MountingHole_3.7mm
- J1, J2: value Conn_01x04_Male -> Conn_01x05; footprint Library:PinHeader_1x04_P2.54mm_Vertical_mirrored -> Samtec:SAMTEC_TSS-105-04-F-S-RA
- JP1: value A3 -> 0
- JP2: value A5 -> 2
- JP3: value A4 -> 1
- JP4: value A6 -> 3
- R1, R10, R11, R12, R13, R14, R15, R16, R17, R18, R19, R2, R20, R21, R22, R23, R24, R3, R4, R5, R6, R7, R8, R9: value 150 -> R_Small_US
- moved J2 201.1 mm to (216.3, 72.4), turned to 180 degrees
- moved J1 165.4 mm to (47.4, 72.4), turned to 180 degrees
- moved C4 111.1 mm to (228.3, 47.4), turned to 0 degrees
- moved R17 68.2 mm to (178.8, 43.3)
- moved R19 61.7 mm to (183.6, 64.0), turned to 90 degrees
- moved R18 56.9 mm to (178.8, 45.7), turned to 0 degrees
- moved H1 56.7 mm to (243.7, 78.6)
- moved H2 56.1 mm to (29.4, 78.6)
- moved R20 55.8 mm to (186.0, 64.0), turned to 90 degrees
- moved R16 55.4 mm to (166.9, 44.1)
- moved R1 53.0 mm to (59.4, 43.4)
- moved R21 51.2 mm to (188.3, 63.9), turned to 90 degrees
- moved R24 49.7 mm to (196.2, 63.9), turned to 90 degrees
- moved R22 48.5 mm to (191.1, 63.9), turned to 90 degrees
- moved R23 47.9 mm to (193.7, 63.9), turned to 90 degrees
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- renumbered DA-0 to D1, DB-1 to D10, DB-2 to D11, DB-3 to D12, DB-4 to D13, DB-5 to D14, DB-6 to D15, DA-1 to D2, DA-2 to D3, DA-3 to D4, DA-4 to D5, DA-5 to D6, DA-6 to D7, DA-7 to D8, DB-0 to D9
Connections:
- C10 pad 1: +5V -> /+5V
- C10 pad 2: GND -> /GND
- C3 pad 1: +5V -> /+5V
- C3 pad 2: GND -> /GND
- C4 pad 1: +5V -> /+5V
- C4 pad 2: GND -> /GND
- C7 pad 1: +5V -> /+5V
- C7 pad 2: GND -> /GND
- D1 pad 1: Net-(DA-0-Pad1) -> /led1
- D1 pad 2: +5V -> /+5V
- D10 pad 1: Net-(DB-1-Pad1) -> /led10
- D10 pad 2: +5V -> /+5V
- D11 pad 1: Net-(DB-2-Pad1) -> /led11
- D11 pad 2: +5V -> /+5V
- D12 pad 1: Net-(DB-3-Pad1) -> /led12
- D12 pad 2: +5V -> /+5V
- D13 pad 1: Net-(DB-4-Pad1) -> /led13
- D13 pad 2: +5V -> /+5V
- D14 pad 1: Net-(DB-5-Pad1) -> /led14
- D14 pad 2: +5V -> /+5V
- D15 pad 1: Net-(DB-6-Pad1) -> /led15
- D15 pad 2: +5V -> /+5V
- D2 pad 1: Net-(DA-1-Pad1) -> /led2
- D2 pad 2: +5V -> /+5V
- D3 pad 1: Net-(DA-2-Pad1) -> /led3
- D3 pad 2: +5V -> /+5V
- D4 pad 1: Net-(DA-3-Pad1) -> /led4
- D4 pad 2: +5V -> /+5V
- D5 pad 1: Net-(DA-4-Pad1) -> /led5
- D5 pad 2: +5V -> /+5V
- D6 pad 1: Net-(DA-5-Pad1) -> /led6
- D6 pad 2: +5V -> /+5V
- D7 pad 1: Net-(DA-6-Pad1) -> /led7
- D7 pad 2: +5V -> /+5V
- D8 pad 1: Net-(DA-7-Pad1) -> /led8
- D8 pad 2: +5V -> /+5V
- D9 pad 1: Net-(DB-0-Pad1) -> /led9
- D9 pad 2: +5V -> /+5V
- J1 pad 1: +5V -> /GND_in1
- J1 pad 2: /SCL -> /GND_in1
- J1 pad 3: /SDA -> /GND_in1
- J1 pad 4: GND -> /+5V_in1
- J2 pad 1: +5V -> /GND
- J2 pad 2: /SCL -> /GND
- J2 pad 3: /SDA -> /GND
- J2 pad 4: GND -> /+5V
- JP1 pad 1: GND -> /GND
- JP1 pad 2: /A3 -> /B0
- JP1 pad 3: +5V -> /+5V
- JP2 pad 1: GND -> /GND
- JP2 pad 2: /A5 -> /B2
- JP2 pad 3: +5V -> /+5V
- JP3 pad 1: GND -> /GND
- JP3 pad 2: /A4 -> /B1
- JP3 pad 3: +5V -> /+5V
- JP4 pad 1: GND -> /GND
- JP4 pad 2: /A6 -> /B3
- JP4 pad 3: +5V -> /+5V
- R1 pad 1: Net-(DA-0-Pad1) -> /led0
- R10 pad 1: Net-(DB-1-Pad1) -> /led9
- R11 pad 1: Net-(DB-2-Pad1) -> /led10
- R12 pad 1: Net-(DB-3-Pad1) -> /led11
- R13 pad 1: Net-(DB-4-Pad1) -> /led12
- R14 pad 1: Net-(DB-5-Pad1) -> /led13
- R15 pad 1: Net-(DB-6-Pad1) -> /led14
- R16 pad 1: Net-(DB-7-Pad1) -> /led15
- R17 pad 1: Net-(DA-P1-Pad1) -> /led16
- R18 pad 1: Net-(DB-P1-Pad1) -> /led17
- R19 pad 1: Net-(DX-0-Pad1) -> /led18
- R2 pad 1: Net-(DA-1-Pad1) -> /led1
- R20 pad 1: Net-(DX-1-Pad1) -> /led19
- R21 pad 1: Net-(DX-2-Pad1) -> /led20
- R22 pad 1: Net-(DX-3-Pad1) -> /led21
- R23 pad 1: Net-(DX-4-Pad1) -> /led22
- R24 pad 1: Net-(DX-5-Pad1) -> /led23
- R3 pad 1: Net-(DA-2-Pad1) -> /led2
- R4 pad 1: Net-(DA-3-Pad1) -> /led3
- R5 pad 1: Net-(DA-4-Pad1) -> /led4
- R6 pad 1: Net-(DA-5-Pad1) -> /led5
- R7 pad 1: Net-(DA-6-Pad1) -> /led6
- R8 pad 1: Net-(DA-7-Pad1) -> /led7
- R9 pad 1: Net-(DB-0-Pad1) -> /led8
- U1 pad 1: +5V -> /B0
- U1 pad 10: GND -> /GND
- U1 pad 15: GND -> /GND
- U1 pad 16: /A5 -> /GND
- U1 pad 17: /A6 -> /GND
- U1 pad 2: GND -> /B1
- U1 pad 20: +5V -> /+5V
- U1 pad 3: GND -> /B2
- U1 pad 4: /A3 -> /B3
- U1 pad 5: /A4 -> /+5V
- U2 pad 1: +5V -> /B0
- U2 pad 10: GND -> /GND
- U2 pad 15: GND -> /GND
- U2 pad 16: /A5 -> /+5V
- U2 pad 17: /A6 -> /GND
- U2 pad 2: +5V -> /B1
- U2 pad 20: +5V -> /+5V
- U2 pad 3: GND -> /B2
- U2 pad 4: /A3 -> /B3
- U2 pad 5: /A4 -> /+5V
- U3 pad 1: +5V -> /B0
- U3 pad 10: GND -> /GND
- U3 pad 15: GND -> /GND
- U3 pad 16: /A5 -> /GND
- U3 pad 17: /A6 -> /+5V
- U3 pad 2: GND -> /B1
- U3 pad 20: +5V -> /+5V
- U3 pad 3: +5V -> /B2
- U3 pad 4: /A3 -> /B3
- U3 pad 5: /A4 -> /+5V
Routing:
- net +5V: track 419.8 -> 0.00 mm, vias 20 -> 0
- net /B0: track 0.00 -> 233.7 mm, vias 0 -> 8
- net /B1: track 0.00 -> 230.2 mm, vias 0 -> 6
- net /B2: track 0.00 -> 143.4 mm, vias 0 -> 4
- net /led0: track 0.00 -> 143.3 mm, vias 0 -> 2
- net /B3: track 0.00 -> 141.2 mm, vias 0 -> 4
- net /led3: track 0.00 -> 133.3 mm, vias 0 -> 2
- net /led1: track 0.00 -> 131.8 mm, vias 0 -> 2
- net /A5: track 131.5 -> 0.00 mm, vias 4 -> 0
- net /A6: track 131.4 -> 0.00 mm, vias 4 -> 0
- net /A3: track 131.0 -> 0.00 mm, vias 4 -> 0
- net /A4: track 130.2 -> 0.00 mm, vias 4 -> 0
- net /led2: track 0.00 -> 126.6 mm, vias 0 -> 2
- net /led7: track 0.00 -> 116.6 mm, vias 0 -> 4
- net /led17: track 0.00 -> 112.3 mm
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- added copper zone on B.Cu, net /+5V
- added copper zone on F.Cu, net /GND
- removed copper zone on B.Cu, net GND
- removed copper zone on F.Cu, net GND
Other:
- board size 221.5 x 18.3 mm -> 222.2 x 57.1 mm
- board text added: "+ gnd: Analog out"
- board text added: "-"
- board text added: "1"
- board text added: "1 0"
- board text added: "ADS7828"
- board text added: "Analog in"
- board text added: "Board select"
- board text added: "LEDs"
- board text added: "MCP47CVB01"
- board text added: "PCA9555D"
- board text added: "Power +5 +5 g g g"
- board text added: "Power in: +5 +5 g g g"
- board text added: "SDA SCL"
- board text added: "System/360 Model 50 console driver Ken Shirriff righto.com/360led v1.2.1"
- board text removed: "SCL"
- board text removed: "SDA"
- board text removed: "System/360 Model 50 console LED driver Ken Shirriff righto.com/s360 v1.0"
