File: hardware/led-driver/led-driver.kicad_sch (KiCad schematic)
At the start: 63 parts, among them J1 Conn_01x04_Male, J2 Conn_01x04_Male, U1 PCA9634, U2 PCA9634, U3 PCA9634

Commit message: Submitted version of board, 1.2.1
Parts:
- removed DX-0, DX-1, DX-2, DX-3, DX-4, DX-5: LED, Library:LED_D3.0mm-nosilk, symbol Device:LED
- removed J1, J2: Conn_01x04_Male, Library:PinHeader_1x04_P2.54mm_Vertical_mirrored, symbol Connector:Conn_01x04_Male
- added C1, C11, C5, C6, C8, C9: .33uF, Capacitor_SMD:C_0805_2012Metric_Pad1.18x1.45mm_HandSolder, symbol Device:C_Small
- added C12: 100uF, Capacitor_Tantalum_SMD:CP_EIA-7343-40_Kemet-Y_Pad2.25x2.55mm_HandSolder, symbol Device:C_Small
- added J1, J2, J6: Conn_01x05, Samtec:SAMTEC_TSS-105-04-F-S-RA, symbol Connector_Generic:Conn_01x05
- added J3: Conn_02x20_Odd_Even, Samtec:SAMTEC_TSS-120-04-F-D-RA-mirror, symbol Connector_Generic:Conn_02x20_Odd_Even
- added J4: Conn_02x25_Odd_Even, Samtec:SAMTEC_TSS-125-04-F-D-RA-mirror, symbol Connector_Generic:Conn_02x25_Odd_Even
- added J5: Conn_01x02, Samtec:SAMTEC_TSS-102-04-F-S-RA, symbol Connector_Generic:Conn_01x02
- added J7: Conn_02x10_Odd_Even, Samtec:SAMTEC_TSS-110-04-F-D-RA-mirror, symbol Connector_Generic:Conn_02x10_Odd_Even
- added J8, J9: Conn_01x02_Male, Samtec:SAMTEC_TSS-102-04-F-S-RA, symbol Connector:Conn_01x02_Male
- added L1, L2: 330 µH, Library:L_Bourns_SDR1307, symbol pspice:INDUCTOR
- added R25: 4.7K, Resistor_SMD:R_0805_2012Metric_Pad1.20x1.40mm_HandSolder, symbol Device:R_Small_US
- added U4, U8: PCA9555D, Package_SO:SOIC-24W_7.5x15.4mm_P1.27mm, symbol Interface_Expansion:PCA9555D
- added U5, U6: ADS7828, Package_SO:TSSOP-16_4.4x5mm_P0.65mm, symbol Analog_ADC:ADS7828
- added U7: MCP47CVB01, Package_SO:MSOP-10_3x3mm_P0.5mm, symbol Library:MCP47CVB01
- C10: renamed from C3; value .1uF -> .33uF
- C3: renamed from C1; value .1uF -> .33uF
- C4: value 10uF -> .33uF
- C7: renamed from C2; value .1uF -> .33uF
- H1, H2: footprint Mounting_Holes:MountingHole_4.3mm_M4 -> MountingHole:MountingHole_3.7mm
- JP1: value A3 -> 0
- JP2: value A5 -> 2
- JP3: value A4 -> 1
- JP4: value A6 -> 3
- R1, R10, R11, R12, R13, R14, R15, R16, R17, R18, R19, R2, R20, R21, R22, R23, R24, R3, R4, R5, R6, R7, R8, R9: value 150 -> R_Small_US
- renumbered DA-0 to D0, DA-1 to D1, DB-2 to D10, DB-3 to D11, DB-4 to D12, DB-5 to D13, DB-6 to D14, DB-7 to D15, DA-2 to D2, DA-3 to D3, DA-4 to D4, DA-5 to D5, DA-6 to D6, DA-7 to D7, DB-0 to D8, DB-1 to D9, DA-P1 to DP0, DB-P1 to DP1
Connections:
- net +5V: now also U1.5 (A4), U2.16 (A5), U2.5 (A4), U3.17 (A6), U3.5 (A4), C1.1, C11.1, C12.1, C6.1, C9.1, J2.4 (Pin_4), J2.5 (Pin_5), J4.1 (Pin_1), J4.11 (Pin_11), J4.13 (Pin_13), J4.15 (Pin_15), J4.17 (Pin_17), J4.19 (Pin_19), J4.21 (Pin_21), J4.23 (Pin_23), J4.25 (Pin_25), J4.27 (Pin_27), J4.29 (Pin_29), J4.3 (Pin_3), J4.31 (Pin_31), J4.33 (Pin_33), J4.35 (Pin_35), J4.37 (Pin_37), J4.39 (Pin_39), J4.41 (Pin_41), J4.43 (Pin_43), J4.45 (Pin_45), J4.47 (Pin_47), J4.49 (Pin_49), J4.5 (Pin_5), J4.7 (Pin_7), J4.9 (Pin_9), J6.4 (Pin_4), J6.5 (Pin_5), J7.2 (Pin_2), J7.20 (Pin_20), L1.2, U4.24 (VDD), U5.13 (A1), U5.16 (VDD), U6.16 (VDD), U7.1 (Vdd), U8.24 (VDD), U8.3 (A2); no longer U1.1 (A0), U2.1 (A0), U2.2 (A1), U3.1 (A0), U3.3 (A2)
- net GND: now also U1.16 (A5), U1.17 (A6), U2.17 (A6), U3.16 (A5), C1.2, C11.2, C12.2, C5.2, C6.2, C8.2, C9.2, J2.1 (Pin_1), J2.2 (Pin_2), J2.3 (Pin_3), J3.1 (Pin_1), J3.2 (Pin_2), J3.3 (Pin_3), J3.37 (Pin_37), J3.38 (Pin_38), J3.39 (Pin_39), J3.4 (Pin_4), J3.40 (Pin_40), J5.1 (Pin_1), J6.1 (Pin_1), J6.2 (Pin_2), J6.3 (Pin_3), J7.1 (Pin_1), J7.19 (Pin_19), L2.2, U4.12 (VSS), U4.3 (A2), U5.11 (COM), U5.9 (GND), U6.11 (COM), U6.13 (A1), U6.9 (GND), U7.6 (~LAT~/HVC), U7.7 (Gnd), U8.12 (VSS); no longer U1.2 (A1), U1.3 (A2), U2.3 (A2), U3.2 (A1)
- net SCL: now also J8.1 (Pin_1), J9.1 (Pin_1), U4.22 (SCL), U5.14 (SCL), U6.14 (SCL), U7.9 (SCL), U8.22 (SCL)
- net SDA: now also J8.2 (Pin_2), J9.2 (Pin_2), U4.23 (SDA), U5.15 (SDA), U6.15 (SDA), U7.10 (SDA), U8.23 (SDA)
- net led0: now reaches D0.1 (K), R1.1
- net led0: now also J4.2 (Pin_2)
- net led1: now reaches D1.1 (K), R2.1
- net led1: now also J4.4 (Pin_4)
- net led2: now reaches D2.1 (K), R3.1
- net led2: now also J4.6 (Pin_6)
- net led3: now reaches D3.1 (K), R4.1
- net led3: now also J4.8 (Pin_8)
- net led4: now reaches D4.1 (K), R5.1
- net led4: now also J4.10 (Pin_10)
- net led5: now reaches D5.1 (K), R6.1
- net led5: now also J4.12 (Pin_12)
- net led6: now reaches D6.1 (K), R7.1
- net led6: now also J4.14 (Pin_14)
- net led7: now reaches D7.1 (K), R8.1
- net led7: now also J4.16 (Pin_16)
- net led15: now reaches D15.1 (K), R16.1
- net led15: now also J4.32 (Pin_32)
- net led14: now reaches D14.1 (K), R15.1
- net led14: now also J4.30 (Pin_30)
- net led13: now reaches D13.1 (K), R14.1
- net led13: now also J4.28 (Pin_28)
- net led12: now reaches D12.1 (K), R13.1
- net led12: now also J4.26 (Pin_26)
- net led11: now reaches D11.1 (K), R12.1
- net led11: now also J4.24 (Pin_24)
- net led10: now reaches D10.1 (K), R11.1
- net led10: now also J4.22 (Pin_22)
- net led9: now reaches D9.1 (K), R10.1
- net led9: now also J4.20 (Pin_20)
- net led8: now reaches D8.1 (K), R9.1
- net led8: now also J4.18 (Pin_18)
- net led23: now reaches R24.1
- net led23: now also J4.48 (Pin_48)
- net led22: now reaches R23.1
- net led22: now also J4.46 (Pin_46)
- net led21: now reaches R22.1
- net led21: now also J4.44 (Pin_44)
- net led20: now reaches R21.1
- net led20: now also J4.42 (Pin_42)
- net led19: now reaches R20.1
- net led19: now also J4.40 (Pin_40)
- net led18: now reaches R19.1
- net led18: now also J4.38 (Pin_38)
- net led17: now reaches DP1.1 (K), R18.1
- net led17: now also J4.36 (Pin_36)
- net led16: now reaches DP0.1 (K), R17.1
- net led16: now also J4.34 (Pin_34)
- net A3 renamed B3
- net B3: now also JP4.2 (C); no longer JP1.2 (C)
- removed net A4: JP3.2 (C), U1.5 (A4), U2.5 (A4), U3.5 (A4)
- removed net A5: JP2.2 (C), U1.16 (A5), U2.16 (A5), U3.16 (A5)
- removed net A6: JP4.2 (C), U1.17 (A6), U2.17 (A6), U3.17 (A6)
- new net: R25.2, U7.4 (Vout)
- new net: C8.1, U6.10 (REF)
- new net: C5.1, U5.10 (REF)
- new net: J5.2 (Pin_2), R25.1
- new net +5V_in1: J1.4 (Pin_4), J1.5 (Pin_5), L1.1
- new net 10a: J3.14 (Pin_14), U4.14 (IO1_1)
- new net 10b: J3.30 (Pin_30), U8.14 (IO1_1)
- new net 11a: J3.15 (Pin_15), U4.15 (IO1_2)
- new net 11b: J3.31 (Pin_31), U8.15 (IO1_2)
- new net 12a: J3.16 (Pin_16), U4.16 (IO1_3)
- new net 12b: J3.32 (Pin_32), U8.16 (IO1_3)
- new net 13a: J3.17 (Pin_17), U4.17 (IO1_4)
- new net 13b: J3.33 (Pin_33), U8.17 (IO1_4)
- new net 14a: J3.18 (Pin_18), U4.18 (IO1_5)
- new net 14b: J3.34 (Pin_34), U8.18 (IO1_5)
- new net 15a: J3.19 (Pin_19), U4.19 (IO1_6)
- new net 15b: J3.35 (Pin_35), U8.19 (IO1_6)
- new net 16a: J3.20 (Pin_20), U4.20 (IO1_7)
- new net 16b: J3.36 (Pin_36), U8.20 (IO1_7)
- new net 1a: J3.5 (Pin_5), U4.4 (IO0_0)
- new net 1b: J3.21 (Pin_21), U8.4 (IO0_0)
- new net 2a: J3.6 (Pin_6), U4.5 (IO0_1)
- new net 2b: J3.22 (Pin_22), U8.5 (IO0_1)
- new net 3a: J3.7 (Pin_7), U4.6 (IO0_2)
- new net 3b: J3.23 (Pin_23), U8.6 (IO0_2)
- new net 4a: J3.8 (Pin_8), U4.7 (IO0_3)
- new net 4b: J3.24 (Pin_24), U8.7 (IO0_3)
- new net 5a: J3.9 (Pin_9), U4.8 (IO0_4)
- new net 5b: J3.25 (Pin_25), U8.8 (IO0_4)
- new net 6a: J3.10 (Pin_10), U4.9 (IO0_5)
- new net 6b: J3.26 (Pin_26), U8.9 (IO0_5)
- new net 7a: J3.11 (Pin_11), U4.10 (IO0_6)
- new net 7b: J3.27 (Pin_27), U8.10 (IO0_6)
- new net 8a: J3.12 (Pin_12), U4.11 (IO0_7)
- new net 8b: J3.28 (Pin_28), U8.11 (IO0_7)
- new net 9a: J3.13 (Pin_13), U4.13 (IO1_0)
- new net 9b: J3.29 (Pin_29), U8.13 (IO1_0)
- new net B0: JP1.2 (C), U1.1 (A0), U2.1 (A0), U3.1 (A0), U4.21 (A0), U5.12 (A0), U6.12 (A0), U7.2 (A0), U8.21 (A0)
- new net B1: JP3.2 (C), U1.2 (A1), U2.2 (A1), U3.2 (A1), U4.2 (A1), U7.8 (A1), U8.2 (A1)
- new net B2: JP2.2 (C), U1.3 (A2), U2.3 (A2), U3.3 (A2)
- new net GND_in1: J1.1 (Pin_1), J1.2 (Pin_2), J1.3 (Pin_3), L2.1
- new net a1a: J7.3 (Pin_3), U6.1 (CH0)
- new net a1b: J7.11 (Pin_11), U5.1 (CH0)
- new net a2a: J7.4 (Pin_4), U6.2 (CH1)
- new net a2b: J7.12 (Pin_12), U5.2 (CH1)
- new net a3a: J7.5 (Pin_5), U6.3 (CH2)
- new net a3b: J7.13 (Pin_13), U5.3 (CH2)
- new net a4a: J7.6 (Pin_6), U6.4 (CH3)
- new net a4b: J7.14 (Pin_14), U5.4 (CH3)
- new net a5a: J7.7 (Pin_7), U6.5 (CH4)
- new net a5b: J7.15 (Pin_15), U5.5 (CH4)
- new net a6a: J7.8 (Pin_8), U6.6 (CH5)
- new net a6b: J7.16 (Pin_16), U5.6 (CH5)
- new net a7a: J7.9 (Pin_9), U6.7 (CH6)
- new net a7b: J7.17 (Pin_17), U5.7 (CH6)
- new net a8a: J7.10 (Pin_10), U6.8 (CH7)
- new net a8b: J7.18 (Pin_18), U5.8 (CH7)
- no-connect marks 0 -> 4
Other:
- note added: "I2C 11000bb"
- note added: "I2C: 01000bb"
- note added: "I2C: 01001bb"
- note added: "I2C: 100100b"
- note added: "I2C: 100101b"
- note added: "I2C: cc1bbbb where cc is the chip 00, 01, 10 and bbbb is the board"
- moved on the sheet: H1, H2
